File: PC-FX/schematics/CD_board/dsp.kicad_sch (KiCad schematic)
At the start: 33 parts, among them CN107 Conn_01x05_Pin, IC102 CXD2500BQ, IC106 CXD1167Q, IC405 74LV08, Q104 Q_NPN_BCE, X101 16.8MHz

Commit message: Progress mainly on SCSI chips and connections to the MCU
Parts:
- removed Q104: Q_NPN_BCE, symbol Device:Q_NPN_BCE
- added C113, C114, C160: ?, Capacitor_SMD:C_0603_1608Metric, symbol Device:C
- added D103: BAT54C, Package_TO_SOT_SMD:SOT-23, symbol Diode:BAT54C
- added unit 3 of IC106
- added unit 2 of IC106
- added Q104: 2N7002, Package_TO_SOT_SMD:SOT-23, symbol SNES:2N7002
- added R110: 3k, symbol Device:R
- added R111: 56k, symbol Device:R
- added R124: 39k, symbol Device:R
- added R125: 33k, symbol Device:R
- added R126: 22k, symbol Device:R
- added R128, R621: ~, symbol Device:R
Connections:
- net +5V: now also C113.2
- net GND: now also C113.1, IC106.4 (V-)
- net VCC: now also IC106.8 (V+)
- net at R129.1: now also C116.2, R127.2, R192.2, IC106.5 (+); no longer IC102.4 (MDP)
- net VC: now reaches C116.1, R127.1
- net VC: now also C161.1, R153.1, Q104.2, R128.2; no longer R129.2, R192.2
- net XTAO: now reaches R163.2
- net at IC405.6: now also Q104.1
- net at R192.1: now also Q104.3
- removed net VC?: C116.2, C161.2, C605.2, R127.2, R153.2
- new net: C161.2, IC106.3 (+), R153.2
- new net: D103.1, R110.1
- new net: IC102.4 (MDP), R129.2
- new net: C160.2, IC106.6 (-), R126.2, R128.1
- new net: C114.2, D103.3, IC106.2 (-), R124.2, R125.1
- new net: D103.2, R111.1
- new net IC106_P7: C160.1, IC106.7, R125.2, R126.1
- new net IC401_PB0: R111.2
- new net IC401_PB1: R110.2
- new net SPO: C114.1, IC106.1, R124.1, R621.1, R621.2
Other:
- note added: "IC104 P10"
- note removed: "IC402 P90"
- moved on the sheet: C116, R127, R129, R153, R192

Commit message: Update on DSP sheet mainly.
Parts:
- removed IC106: CXD1167Q, Package_QFP:PQFP-100_14x20mm_P0.65mm, symbol PC-Engine_CDR-30:CXD1167Q
- removed L102: L, symbol Device:L
- removed R500, R503, R504, R529, R532: 220, Resistor_SMD:R_0603_1608Metric, symbol Device:R
- removed R528: 0, Resistor_SMD:R_0603_1608Metric, symbol Device:R
- removed R531: 100, Resistor_SMD:R_0603_1608Metric, symbol Device:R
- removed R537: 10k, Resistor_SMD:R_0603_1608Metric, symbol Device:R
- added C1: 100uF, Capacitor_SMD:CP_Elec_5x5.4, symbol Device:C_Polarized
- added C110, C127, C140, C141, C151, C157, C159, C162, C163: ?, symbol Device:C
- added C119, C121, C149: ?, Capacitor_SMD:C_0603_1608Metric, symbol Device:C
- added C126, C142: 47uF, Capacitor_SMD:CP_Elec_5x5.4, symbol Device:C_Polarized
- added C147, C153, C154, C156: C, symbol Device:C
- added C152: 4.7uF, Capacitor_SMD:CP_Elec_5x5.4, symbol Device:C_Polarized
- added IC109: BA7082F, Package_SO:SOIC-16_4.55x10.3mm_P1.27mm, symbol PC-FX:BA7082F
- added IC110: 74AHC1G04, symbol 74xGxx:74AHC1G04
- added unit 3 of IC405
- added IC406: 74LV04, symbol PC-FX:74LV04
- added R131, R134, R161, R163, R169: 10k, symbol Device:R
- added R132: 6k8, symbol Device:R
- added R133: 3k3, symbol Device:R
- added R135: 100k, symbol Device:R
- added R162, R165: 120k, symbol Device:R
- added R164: 3k9, symbol Device:R
- added R167: 100, symbol Device:R
- added R168: 5k1, symbol Device:R
- added R172: 33k, symbol Device:R
- added R173, R175, R178, R179, R180, R181, R182: ~, symbol Device:R
- added R174: 47k, symbol Device:R
- added TP101: VCO, symbol Connector:TestPoint
- added TP140: TestPoint, symbol Connector:TestPoint
- added VR106: R_Potentiometer, Potentiometer_THT:Potentiometer_Bourns_3339P_Vertical, symbol Device:R_Potentiometer
Connections:
- net MD2 is gone; now on net GND: IC102.59 (MD2)
- net +5V: now also C110.1, C141.2, C142.1, C147.1, C154.1, C156.1, IC109.10 (VCC), R161.1, R174.1, R182.2
- net GND: now also IC102.10 (TEST), IC102.25 (BIAS), IC102.26 (ASYI), IC102.28 (ASYE), IC102.30 (PSSL), IC102.9 (VCOI), C1.2, C110.2, C121.2, C126.2, C127.2, C142.2, C147.2, C152.2, C153.2, C154.2, C156.2, C159.2, C162.2, C163.1, C163.2, IC109.6 (1/2FB), IC109.8 (GND), IC110.3 (GND), R163.2, R168.2, R169.2, R173.2, R180.2, R181.1, R181.2, R182.1, VR106.1, VR106.2
- net LOCK: now also IC102.6 (LOCK), IC405.5
- net MDP: now also IC102.4 (MDP), R129.2
- net MRST: now also IC102.70 (XRST)
- net SBSO: now also IC406.6; no longer IC102.64 (SBSO)
- net VCC: now also IC110.5 (VCC)
- net IC103_P25: now reaches C128.1, R137.2
- net IC103_P25: no longer IC102.70 (XRST)
- net VPCO: now reaches IC102.16 (VPCO)
- net VPCO: now also R161.2, R162.2, R163.1
- net VCKI: now reaches IC102.17 (VCKI)
- net VCKI: now also R167.2, TP140.1
- net FILO: now reaches IC102.18 (FILO)
- net FILO: now also C140.2, R134.1
- net FILI: now reaches IC102.19 (FILI)
- net FILI: now also R132.2, R133.1
- net PCO: now reaches IC102.20 (PCO)
- net PCO: now also R132.1
- net CLTV: now reaches IC102.22 (CLTV)
- net CLTV: now also C141.1, R134.2
- net IC103_P32: now reaches IC102.24 (RF)
- net IC103_P32: now also C149.1, C149.2, R175.2, R178.1, R178.2
- net at IC102.27 (ASYO): now also R131.2, R179.2
- net APTL: no longer names the net of IC102.51 (APTL)
- net APTR: no longer names the net of IC102.50 (APTR)
- net BCLK renamed DSP_BCLK
- net C4M: no longer names the net of IC102.57 (C4M)
- net DOUT renamed DSP_DOUT
- net FSTT: no longer names the net of IC102.56 (FSTT)
- net LRCK renamed DSP_LRCK
- net WDCK renamed DSP_WDCK
- new net: C162.1, R179.1, R180.1
- new net: C151.1, IC109.11 (CT2)
- new net: C151.2, IC109.12 (CT1)
- new net: IC405.9, IC406.8
- new net: C140.1, R133.2
- new net: IC109.15 (IN2), R165.1
- new net: IC109.13 (VCTL), IC109.14 (VO), R165.2, TP101.1
- new net: C127.1, R131.1, R135.2
- new net: C152.1, C153.1, IC109.16 (IN1), R162.1, R164.1
- new net: C157.2, IC110.2, R169.1
- new net: IC110.4, R167.1
- new net: IC405.10, IC406.4
- new net: IC405.8, IC406.5
- new net: C157.1, IC109.7 (FOUT), R168.1
- new net: C1.1, R164.2
- new net: C159.1, R172.1, R173.1, VR106.3
- new net: IC109.9 (FADJ), R172.2
- new net: IC109.4 (BW), IC109.5 (BWB), R174.2
- new net DSP_SBSO: IC102.64 (SBSO), IC406.9
- new net IC103_P31: C126.1, R135.1
- new net IC103_P39: C119.2
- new net IC103_P40: C119.1, R175.1
- new net IC103_P44: C121.1
- new net ~{LDON}: IC406.3
- no-connect marks 15 -> 23
Other:
- note added: "CN401 P13"
- note added: "IC101 P19"
- note added: "IC102 P16 (VPCO)"
- note added: "IC102 P17 (VCKI)"
- note added: "MD2='0' => DOUT is off"
- note added: "SUBCODE: SCOR is block sync WFCK is frame sync SBSO is data out EXCK is external clock (from PC-FX main board)"
- note added: "SUBQCODE: SQCK is clock SQSO is data out"
- note added: "VR106 FADJ"
- note removed: "CDR-30 (older revision used CXD1135 with external RAM IC107 HM6116 instead but seemed to be the same). CXD1167 must have built in RAM - Edit: some CDR-30As also come with CXD1135 + RAM"
- note removed: "GFS is the output of the lock conditions of frame sync"
- note removed: "IC103 P25"
- note removed: "IC202 P9"
- note removed: "IOs connected to micro IC 108 SQCK is an input when SQEX=H All subcode Q related signals 2 possible modes: "10000" (normal audio) where XIN = 8MHz, Digital filter is ON, audio is send via serial output Audio cata is always using 2's complement output format "11101"(test mode as far as I can tell), with DF off, parallel data, 2's perhaps an undefined CD ROM mode as not listed in KS5990 datasheet"
- note removed: "R528 to R536 do not exist on the older revision CRD-30"
- note removed: "Spindle servo connections to CXA1082"
- note removed: "To IFU connector on pin A6"
- note removed: "To IFU connector on pin B4, A12, A14 SBSY (Block synchronization) connected to micro's interrupt input SBCK comes from IFU PW is Subcode data P to W (8-bits)"
- moved on the sheet: C113, C114, C116, C128, C140, C141, C142, C143, C160, C161, C605, CN107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

Commit message: Schematics pretty much done. Expect some mistakes but it captures enough information to help understanding its behaviour.
Parts:
- removed C113, C114, C116, C119, C121, C149, C160, C161, C605: ?, Capacitor_SMD:C_0603_1608Metric, symbol Device:C
- removed C142, C143: 100nF, Capacitor_SMD:C_0603_1608Metric, symbol Device:C
- removed D103: BAT54C, Package_TO_SOT_SMD:SOT-23, symbol Diode:BAT54C
- removed IC106: BA4510F, Package_SO:SSOP-8_5.25x5.24mm_P1.27mm, symbol PC-FX:BA4510F
- removed unit 2 of IC405
- removed Q104: 2N7002, Package_TO_SOT_SMD:SOT-23, symbol SNES:2N7002
- removed R110: 3k, symbol Device:R
- removed R111: 56k, symbol Device:R
- removed R124, R129: 39k, symbol Device:R
- removed R125: 33k, symbol Device:R
- removed R126: 22k, symbol Device:R
- removed R127: 120k, symbol Device:R
- removed R128, R175, R178, R621: ~, symbol Device:R
- removed R153: 20k, symbol Device:R
- removed R192: 68k, symbol Device:R
- renumbered R179 to R158
Connections:
- net GND: now also R158.2; no longer R158.1
- net SERVO_SENS: now reaches IC102.75 (SEIN)
- net DATO: now reaches IC102.77 (DATO)
- net XLTO: now reaches IC102.78 (XLTO)
- net CLKO: now reaches IC102.79 (CLKO)
- net MIRR: now reaches IC102.80 (MIRR)
- net C.OUT: now reaches R130.1
- net IC103_P25 renamed ~{SERVO_RST}
- net IC103_P31 renamed ASY
- net IC103_P32 renamed EFM
- net MRST renamed ~{MRST}
- net XTSL: no longer names the net of IC102.55 (XTSL)
- net XTSL: now also R158.1; no longer R158.2
Other:
- note added: "MD2 tied to GND => DOUT is off"
- note added: "XTSL Pulled low for 16.9344MHz crystal"
- note removed: "Double speed - IC402 P24 and IC202 P28"
- note removed: "IC103 P22"
- note removed: "IC103 P23"
- note removed: "IC103 P24"
- note removed: "IC103 P26"
- note removed: "IC103 P27"
- note removed: "IC103 P29"
- note removed: "IC104 P10"
- note removed: "MD2='0' => DOUT is off"
- note removed: "Pulled low for 16.9344MHz crystal"
- title: PC FX Pots Adfustment Schematics -> PC-FX CD Board Schematics
- moved on the sheet: C1, C110, C126, C127, C128, C140, C141, C142, C147, C151, C152, C153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

Commit message: Confirmed connections and fixed issues on Servo and DSP chips using similar design - Sony CDP-790
Parts:
- removed C1: 100uF, Capacitor_SMD:CP_Elec_5x5.4, symbol Device:C_Polarized
- added C158: ?, Capacitor_SMD:CP_Elec_5x5.4, symbol Device:C_Polarized
- C153: value C -> ?
Connections:
- net GND: now also C158.2
- net at C153.1, IC109.16 (IN1), R162.1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: now also C158.1; no longer C152.1
- net at R164.2: now also C152.1
- net MNT3: now reaches CN107.4 (Pin_4), IC102.46 (DA04)
- net MNT2: now reaches CN107.3 (Pin_3), IC102.47 (DA03)
- net MNT1: now reaches CN107.2 (Pin_2), IC102.48 (DA02)
- net MNT0: now reaches CN107.1 (Pin_1), IC102.49 (DA01)
Other:
- moved on the sheet: C110, C126, C127, C140, C141, C142, C152, C153, C162, C163, R131, R132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
