File: PC-FX/schematics/CD_board/pcm.kicad_sch (KiCad schematic)
At the start: 27 parts, among them IC201 PCM1710U, IC202 74HC132, IC301 LM7805_TO220, Q201 2N7002

Commit message: Update on DSP sheet mainly.
Parts:
- added C305: 470uF, Capacitor_SMD:CP_Elec_5x5.4, symbol Device:C_Polarized
- added C306: ?, Capacitor_SMD:C_0603_1608Metric, symbol Device:C
Connections:
- net IC403_P90 is gone; now on net DOUT: R171.7 (R2.2)
- net IC403_P91 is gone; now on net BCLK: R171.8 (R1.2)
- net IC403_P92 is gone; now on net WDCK: R171.5 (R4.2)
- net IC403_P94 is gone; now on net LRCK: R171.6 (R3.2)
- net +12V: now also C306.2
- net +5V: now also C305.1
- net BCLK: no longer R171.1 (R1.1), R203.2
- net DOUT: no longer R171.2 (R2.1), R202.1
- net GND: now also C305.2, C306.1
- net LRCK: no longer R171.3 (R3.1), R201.2
- net WDCK: no longer R171.4 (R4.1)
- new net DSP_BCLK: R171.1 (R1.1), R203.2
- new net DSP_DOUT: R171.2 (R2.1), R202.1
- new net DSP_LRCK: R171.3 (R3.1), R201.2
- new net DSP_WDCK: R171.4 (R4.1)

Commit message: Schematics pretty much done. Expect some mistakes but it captures enough information to help understanding its behaviour.
Parts:
- removed C304, C305: 470uF, Capacitor_SMD:CP_Elec_5x5.4, symbol Device:C_Polarized
- removed C306: ?, Capacitor_SMD:C_0603_1608Metric, symbol Device:C
- removed C307: 100uF, Capacitor_SMD:CP_Elec_5x5.4, symbol Device:C_Polarized
- removed IC301: LM7805_TO220, Package_TO_SOT_THT:TO-220-3_Vertical, symbol Regulator_Linear:LM7805_TO220
Other:
- title: PC FX Pots Adfustment Schematics -> PC-FX CD Board Schematics
