File: PC-FX/schematics/CD_board/power.kicad_sch (KiCad schematic)
At the start: 12 parts, among them CN302 Conn_01x04_Pin, IC301 LM7805_TO220

Commit message: Crystal frequency added + PDF of the schematics
Connections:
- net +12V renamed +9V
