File: PC-FX/schematics/CD_board/servo.kicad_sch (KiCad schematic)
At the start: 103 parts, among them CN102 Conn_01x10_Pin, CN104 Conn_01x06_Pin, IC103 CXA1372BQ, IC104 BA6398FP, IC106 BA4510F, IC108 BA4510F, IC405 74LV08, Q104 2N7002, Q106 2N7002

Commit message: Confirmed connections and fixed issues on Servo and DSP chips using similar design - Sony CDP-790
Parts:
- added C129: 1uF, Capacitor_SMD:CP_Elec_5x5.4, symbol Device:C_Polarized
- added C150: 2.2uF, Capacitor_SMD:CP_Elec_5x5.4, symbol Device:C_Polarized
Connections:
- net AVCC: now also C150.1
- net GND: now also C129.2; no longer C121.1
- net SL+: now also C136.2, R144.2; no longer R145.2
- net SL-: now also C112.1, C139.2, D102.1, R148.2, R150.2, R151.1, R196.2; no longer C139.1, Q106.2, R148.1
- net SLO: now also C139.1, Q106.2, R148.1, R155.2
- net VC: now also C121.1, C129.1, C150.2
- net at C112.2, C115.2, Q106.3: now also R196.1; no longer R196.2
- net FZC: no longer names the net of C108.2, IC103.46 (FZC), R115.1
- net TZC: no longer names the net of C120.1, IC103.42 (TZC)
- new net: C137.2, R145.2
Other:
- note added: "External opamps (IC106 and IC108) used to drive the motor H-bridge controller instead of using internal opamps. More flexibility?"
- note added: "Servo controls stopped when FOK = 0 from DSP or when RFO is not present from RF amp"
- note added: "Spindle control comes from DSP chip via MDP pin"
- note added: "fast sled?"
- moved on the sheet: C112, C115, C121, C123, C132, C136, C137, C139, C603, C605, D102, L105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

Commit message: Small update based on confirmation of SCSI control signals
Changed lines of the file:
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@@
 	)
 	(hierarchical_label "ENDSW_A"
-		(shape input)
+		(shape output)
 		(at 210.82 229.87 180)
 		(fields_autoplaced yes)

Commit message: Crystal frequency added + PDF of the schematics
Connections:
- net +12V renamed +9V
Changed lines of the file:
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@@
 	(title_block
 		(title "PC-FX CD Board Schematics")
-		(date "2024-07-21")
+		(date "2024-07-25")
 		(rev "0.1")
 		(company "Author: Regis Galland")
@@
 	)
 	(symbol
+		(lib_id "power:+9V")
+		(at 181.61 181.61 0)
+		(unit 1)
+		(exclude_from_sim no)
+		(in_bom yes)
+		(on_board yes)
+		(dnp no)
+		(fields_autoplaced yes)
+		(property "Reference" "#PWR0128"
+			(at 181.61 185.42 0)
+			(effects
+				(font
+					(size 1.27 1.27)
+				)
+				(hide yes)
+			)
+		)
+		(property "Value" "+9V"
+			(at 181.61 177.4769 0)
+			(effects
+				(font
+					(size 1.27 1.27)
+				)
+			)
+		)
+		(property "Footprint" ""
+			(at 181.61 181.61 0)
+			(effects
+				(font
+					(size 1.27 1.27)
+				)
+				(hide yes)
+			)
+		)
+		(property "Datasheet" ""
+			(at 181.61 181.61 0)
+			(effects
+				(font
+					(size 1.27 1.27)
+				)
+				(hide yes)
+			)
+		)
+		(property "Description" "Power symbol creates a global label with name \"+9V\""
+			(at 181.61 181.61 0)
+			(effects
+				(font
+					(size 1.27 1.27)
+				)
+				(hide yes)
+			)
+		)
+		(pin "1"
+		)
+		(instances
+			(project "CD_board"
+				(path "/28d2c364-a4dd-4270-9fde-bb67593159d8/ebb3f727-b892-4f06-bc76-9637dbfdc33d"
+					(reference "#PWR0128")
+					(unit 1)
+				)
+			)
+		)
+	)
+	(symbol
 		(lib_id "Device:R")
 		(at 285.75 60.96 0)
@@
 	)
 	(symbol
+		(lib_id "power:+9V")
+		(at 219.71 190.5 0)
+		(unit 1)
+		(exclude_from_sim no)
+		(in_bom yes)
+		(on_board yes)
+		(dnp no)
+		(fields_autoplaced yes)
+		(property "Reference" "#PWR088"
+			(at 219.71 194.31 0)
+			(effects
+				(font
+					(size 1.27 1.27)
+				)
+				(hide yes)
+			)
+		)
+		(property "Value" "+9V"
+			(at 219.71 186.3669 0)
+			(effects
+				(font
+					(size 1.27 1.27)
+				)
+			)
+		)
+		(property "Footprint" ""
+			(at 219.71 190.5 0)
+			(effects
+				(font
+					(size 1.27 1.27)
+				)
+				(hide yes)
+			)
+		)
+		(property "Datasheet" ""
+			(at 219.71 190.5 0)
+			(effects
+				(font
+					(size 1.27 1.27)
+				)
+				(hide yes)
+			)
+		)
+		(property "Description" "Power symbol creates a global label with name \"+9V\""
+			(at 219.71 190.5 0)
+			(effects
+				(font
+					(size 1.27 1.27)
+				)
+				(hide yes)
+			)
+		)
+		(pin "1"
+		)
+		(instances
+			(project "CD_board"
+				(path "/28d2c364-a4dd-4270-9fde-bb67593159d8/ebb3f727-b892-4f06-bc76-9637dbfdc33d"
+					(reference "#PWR088")
+					(unit 1)
+				)
+			)
+		)
+	)
+	(symbol
 		(lib_id "Device:C")
 		(at 128.27 256.54 270)
@@
 	)
 	(symbol
-		(lib_id "power:+12V")
-		(at 219.71 190.5 0)
-		(unit 1)
-		(exclude_from_sim no)
-		(in_bom yes)
-		(on_board yes)
-		(dnp no)
-		(fields_autoplaced yes)
-		(property "Reference" "#PWR0130"
-			(at 219.71 194.31 0)
-			(effects
-				(font
-					(size 1.27 1.27)
-				)
-				(hide yes)
-			)
-		)
-		(property "Value" "+12V"
-			(at 219.71 186.3669 0)
-			(effects
-				(font
-					(size 1.27 1.27)
-				)
-			)
-		)
-		(property "Footprint" ""
-			(at 219.71 190.5 0)
-			(effects
-				(font
-					(size 1.27 1.27)
-				)
-				(hide yes)
-			)
-		)
-		(property "Datasheet" ""
-			(at 219.71 190.5 0)
-			(effects
-				(font
-					(size 1.27 1.27)
-				)
-				(hide yes)
-			)
-		)
-		(property "Description" "Power symbol creates a global label with name \"+12V\""
-			(at 219.71 190.5 0)
-			(effects
-				(font
-					(size 1.27 1.27)
-				)
-				(hide yes)
-			)
-		)
-		(pin "1"
-		)
-		(instances
-			(project "CD_board"
-				(path "/28d2c364-a4dd-4270-9fde-bb67593159d8/ebb3f727-b892-4f06-bc76-9637dbfdc33d"
-					(reference "#PWR0130")
-					(unit 1)
-				)
-			)
-		)
-	)
-	(symbol
 		(lib_id "power:GND")
 		(at 231.14 205.74 0)
@@
 	)
 	(symbol
-		(lib_id "Device:R")
-		(at 295.91 52.07 90)
-		(mirror x)
+		(lib_id "power:+9V")
+		(at 166.37 181.61 0)
 		(unit 1)
 		(exclude_from_sim no)
@@
 		(on_board yes)
 		(dnp no)
-		(property "Reference" "R106"
-			(at 293.37 48.006 90)
+		(fields_autoplaced yes)
+		(property "Reference" "#PWR063"
+			(at 166.37 185.42 0)
 			(effects
 				(font
 					(size 1.27 1.27)
 				)
-				(justify right)
+				(hide yes)
 			)
 		)
-		(property "Value" "47k"
-			(at 294.132 50.038 90)
+		(property "Value" "+9V"
+			(at 166.37 177.4769 0)
 			(effects
 				(font
 					(size 1.27 1.27)
 				)
-				(justify right)
 			)
 		)
 		(property "Footprint" ""
-			(at 295.91 50.292 90)
+			(at 166.37 181.61 0)
 			(effects
 				(font
@@
 			)
 		)
-		(property "Datasheet" "~"
-			(at 295.91 52.07 0)
+		(property "Datasheet" ""
+			(at 166.37 181.61 0)
 			(effects
 				(font
@@
 			)
 		)
-		(property "Description" ""
-			(at 295.91 52.07 0)
+		(property "Description" "Power symbol creates a global label with name \"+9V\""
+			(at 166.37 181.61 0)
 			(effects
 				(font
@@
 			)
 		)
-		(pin "2"
-		)
 		(pin "1"
 		)
 		(instances
-			(project "CD_board"
+			(project ""
 				(path "/28d2c364-a4dd-4270-9fde-bb67593159d8/ebb3f727-b892-4f06-bc76-9637dbfdc33d"
-					(reference "R106")
+					(reference "#PWR063")
 					(unit 1)
 				)
@@
 	)
 	(symbol
-		(lib_id "power:+12V")
-		(at 181.61 181.61 0)
+		(lib_id "Device:R")
+		(at 295.91 52.07 90)
+		(mirror x)
 		(unit 1)
 		(exclude_from_sim no)
@@
 		(on_board yes)
 		(dnp no)
-		(fields_autoplaced yes)
-		(property "Reference" "#PWR0129"
-			(at 181.61 185.42 0)
+		(property "Reference" "R106"
+			(at 293.37 48.006 90)
 			(effects
 				(font
 					(size 1.27 1.27)
 				)
-				(hide yes)
+				(justify right)
 			)
 		)
-		(property "Value" "+12V"
-			(at 181.61 177.4769 0)
+		(property "Value" "47k"
+			(at 294.132 50.038 90)
 			(effects
 				(font
 					(size 1.27 1.27)
 				)
+				(justify right)
 			)
 		)
 		(property "Footprint" ""
-			(at 181.61 181.61 0)
+			(at 295.91 50.292 90)
 			(effects
 				(font
@@
 			)
 		)
-		(property "Datasheet" ""
-			(at 181.61 181.61 0)
+		(property "Datasheet" "~"
+			(at 295.91 52.07 0)
 			(effects
 				(font
@@
 			)
 		)
-		(property "Description" "Power symbol creates a global label with name \"+12V\""
-			(at 181.61 181.61 0)
+		(property "Description" ""
+			(at 295.91 52.07 0)
 			(effects
 				(font
@@
 			)
 		)
+		(pin "2"
+		)
 		(pin "1"
 		)
@@
 			(project "CD_board"
 				(path "/28d2c364-a4dd-4270-9fde-bb67593159d8/ebb3f727-b892-4f06-bc76-9637dbfdc33d"
-					(reference "#PWR0129")
+					(reference "R106")
 					(unit 1)
 				)
@@
 					(unit 1)
 				)
-			)
-		)
-	)
-	(symbol
-		(lib_id "power:+12V")
-		(at 166.37 181.61 0)
-		(unit 1)
-		(exclude_from_sim no)
-		(in_bom yes)
-		(on_board yes)
-		(dnp no)
-		(fields_autoplaced yes)
-		(property "Reference" "#PWR0128"
-			(at 166.37 185.42 0)
-			(effects
-				(font
-					(size 1.27 1.27)
-				)
-				(hide yes)
-			)
-		)
-		(property "Value" "+12V"
-			(at 166.37 177.4769 0)
-			(effects
-				(font
-					(size 1.27 1.27)
-				)
-			)
-		)
-		(property "Footprint" ""
-			(at 166.37 181.61 0)
-			(effects
-				(font
-					(size 1.27 1.27)
-				)
-				(hide yes)
-			)
-		)
-		(property "Datasheet" ""
-			(at 166.37 181.61 0)
-			(effects
-				(font
-					(size 1.27 1.27)
-				)
-				(hide yes)
-			)
-		)
-		(property "Description" "Power symbol creates a global label with name \"+12V\""
-			(at 166.37 181.61 0)
-			(effects
-				(font
-					(size 1.27 1.27)
-				)
-				(hide yes)
-			)
-		)
-		(pin "1"
-		)
-		(instances
-			(project "CD_board"
-				(path "/28d2c364-a4dd-4270-9fde-bb67593159d8/ebb3f727-b892-4f06-bc76-9637dbfdc33d"
-					(reference "#PWR0128")
-					(unit 1)
-				)
